File: KiCad/Versie2/arduino_uno_r3_from_scratch-master/voltage_management.sch (KiCad schematic (older format))
At the start: 3 parts, among them U3 LP2985-33DBVR

Commit message: 28feb
Aanpassing KiCad+deel footprints
Changed lines of the file:
@@
 	7800 4200 8000 4200
 Wire Wire Line
-	8000 4000 8000 4200
-Wire Wire Line
-	8000 4200 8000 4450
+	8000 4000 8000 4450
 Wire Wire Line
 	8000 4750 8000 5325
@@
 $EndComp
 Wire Wire Line
-	5400 4200 5650 4200
-Wire Wire Line
-	5650 4200 5900 4200
-Wire Wire Line
-	5900 4200 6200 4200
+	5400 4200 6200 4200
 Text GLabel 8000 4000 0    60   Input ~ 0
 3V3_LDO
