File: KiCad/latestkicadproject/arduino_uno_r3_from_scratch-master/Motor Outputs.sch (KiCad schematic (older format))
At the start: 9 parts, among them X1 DG3XX-04-3.5

Commit message: verbeteringen kicad
Changed lines of the file:
@@
 Comment4 ""
 $EndDescr
-$Comp
-L GND #PWR010
-U 1 1 5A0B3F5C
-P 5100 4700
-F 0 "#PWR010" H 5100 4450 50  0001 C CNN
-F 1 "GND" H 5100 4550 50  0000 C CNN
-F 2 "" H 5100 4700 50  0001 C CNN
-F 3 "" H 5100 4700 50  0001 C CNN
-	1    5100 4700
-	1    0    0    -1
-$EndComp
-$Comp
-L GND #PWR011
-U 1 1 5A0B3F8E
-P 5450 4700
-F 0 "#PWR011" H 5450 4450 50  0001 C CNN
-F 1 "GND" H 5450 4550 50  0000 C CNN
-F 2 "" H 5450 4700 50  0001 C CNN
-F 3 "" H 5450 4700 50  0001 C CNN
-	1    5450 4700
-	1    0    0    -1
-$EndComp
-$Comp
-L GND #PWR012
-U 1 1 5A0B3FB1
-P 5700 4700
-F 0 "#PWR012" H 5700 4450 50  0001 C CNN
-F 1 "GND" H 5700 4550 50  0000 C CNN
-F 2 "" H 5700 4700 50  0001 C CNN
-F 3 "" H 5700 4700 50  0001 C CNN
-	1    5700 4700
-	1    0    0    -1
-$EndComp
-$Comp
-L GND #PWR013
-U 1 1 5A0B43FA
-P 6000 4700
-F 0 "#PWR013" H 6000 4450 50  0001 C CNN
-F 1 "GND" H 6000 4550 50  0000 C CNN
-F 2 "" H 6000 4700 50  0001 C CNN
-F 3 "" H 6000 4700 50  0001 C CNN
-	1    6000 4700
-	1    0    0    -1
-$EndComp
 Wire Wire Line
 	4650 4000 6200 4000
@@
 Wire Wire Line
 	6000 4700 6000 4350
+Text HLabel 5100 4700 0    60   Input ~ 0
+GND
+Text HLabel 5450 4700 0    60   Input ~ 0
+GND
+Text HLabel 5700 4700 0    60   Input ~ 0
+GND
+Text HLabel 6000 4700 0    60   Input ~ 0
+GND
 $EndSCHEMATC
