File: KiCad/latestkicadproject/arduino_uno_r3_from_scratch-master/Driver.sch (KiCad schematic (older format))
At the start: 6 parts, among them U3 74AHC1G04, U4 74AHC1G04, U9 L298

Commit message: PCB routing v1
Parts:
- removed U9: L298, L298P:SOIC127P1420X360-21N, symbol L298
- added IC3: L298P, L298Poud:SOIC127P1420X360-21N, symbol L298P
- C1, C8: footprint Capacitor_SMD:C_0805_2012Metric -> Capacitors_SMD:C_0805
- C7: footprint Capacitors_SMD:C_0805_HandSoldering -> Capacitors_SMD:CP_Elec_6.3x5.3
Connections:
- net +5V: now also IC3.12 (VSS)
- net DIRA: now also IC3.7 (INPUT1)
- net DIRB: now also IC3.13 (INPUT3)
- net GND: now also IC3.1 (GND), IC3.10 (GND_1), IC3.11 (GND_2), IC3.19 (SENSE_B), IC3.2 (SENSE_A), IC3.20 (GND_3), IC3.21 (EP)
- net OUT1: now also IC3.4 (OUT1)
- net OUT2: now also IC3.5 (OUT2)
- net OUT3: now also IC3.16 (OUT3)
- net OUT4: now also IC3.17 (OUT4)
- net PWMA: now also IC3.8 (ENABLE_A)
- net PWMB: now also IC3.14 (ENABLE_B)
- net PWRIN: now also IC3.6 (VS)
- net at U4.4: now also IC3.15 (INPUT4)
- net at U3.4: now also IC3.9 (INPUT2)
Changed lines of the file:
@@
 LIBS:degson
 LIBS:PHT6NQ10T_135
+LIBS:L298P
 EELAYER 25 0
 EELAYER END
@@
 $EndDescr
 $Comp
-L GND #PWR015
+L GND #PWR018
 U 1 1 5A0B4BA1
 P 4250 3300
-F 0 "#PWR015" H 4250 3050 50  0001 C CNN
+F 0 "#PWR018" H 4250 3050 50  0001 C CNN
 F 1 "GND" H 4250 3150 50  0000 C CNN
 F 2 "" H 4250 3300 50  0001 C CNN
@@
 	1    0    0    -1
 $EndComp
-Wire Wire Line
-	4400 2200 4250 2200
-Wire Wire Line
-	4400 2300 4250 2300
-Connection ~ 4250 2300
-Wire Wire Line
-	4400 3100 4250 3100
-Connection ~ 4250 3100
-$Comp
-L GND #PWR016
+$Comp
+L GND #PWR019
 U 1 1 5A0B4C37
 P 6250 3300
-F 0 "#PWR016" H 6250 3050 50  0001 C CNN
+F 0 "#PWR019" H 6250 3050 50  0001 C CNN
 F 1 "GND" H 6250 3150 50  0000 C CNN
 F 2 "" H 6250 3300 50  0001 C CNN
@@
 	1    0    0    -1
 $EndComp
-Wire Wire Line
-	6250 3300 6250 2200
-Wire Wire Line
-	6250 2200 6100 2200
-Wire Wire Line
-	6100 2300 6250 2300
-Connection ~ 6250 2300
-Wire Wire Line
-	6100 3100 6250 3100
-Connection ~ 6250 3100
-Wire Wire Line
-	6100 2500 6650 2500
-Wire Wire Line
-	6100 2600 6825 2600
 Text Label 6350 2500 0    60   ~ 0
 OUT4
 Text Label 6350 2600 0    60   ~ 0
 OUT3
-Wire Wire Line
-	6100 2800 6825 2800
-Wire Wire Line
-	6100 2900 6675 2900
 Text Label 6350 2800 0    60   ~ 0
 PWMB
 Text Label 6350 2900 0    60   ~ 0
 DIRB
-Wire Wire Line
-	6100 3000 6300 3000
-Wire Wire Line
-	6300 3000 6300 2050
 $Comp
 L 74AHC1G04 U4
@@
 	-1   0    0    1
 $EndComp
-Wire Wire Line
-	6100 2700 6650 2700
-$Comp
-L GND #PWR017
+$Comp
+L GND #PWR020
 U 1 1 5A0B4D89
-P 7150 2500
-F 0 "#PWR017" H 7150 2250 50  0001 C CNN
-F 1 "GND" H 7150 2350 50  0000 C CNN
-F 2 "" H 7150 2500 50  0001 C CNN
-F 3 "" H 7150 2500 50  0001 C CNN
-	1    7150 2500
+P 7150 2450
+F 0 "#PWR020" H 7150 2200 50  0001 C CNN
+F 1 "GND" H 7150 2300 50  0000 C CNN
+F 2 "" H 7150 2450 50  0001 C CNN
+F 3 "" H 7150 2450 50  0001 C CNN
+	1    7150 2450
 	-1   0    0    1
 $EndComp
-Wire Wire Line
-	7150 2900 7150 3100
-Wire Wire Line
-	7150 3050 7350 3050
-Connection ~ 7150 3050
 $Comp
 L C C8
@@
 F 0 "C8" H 7525 3150 50  0000 L CNN
 F 1 "0.1uF" H 7525 2950 50  0000 L CNN
-F 2 "Capacitor_SMD:C_0805_2012Metric" H 7538 2900 50  0001 C CNN
+F 2 "Capacitors_SMD:C_0805" H 7538 2900 50  0001 C CNN
 F 3 "" H 7500 3050 50  0001 C CNN
 	1    7500 3050
@@
 $EndComp
 $Comp
-L GND #PWR018
+L GND #PWR021
 U 1 1 5A0B5004
 P 7650 3050
-F 0 "#PWR018" H 7650 2800 50  0001 C CNN
+F 0 "#PWR021" H 7650 2800 50  0001 C CNN
 F 1 "GND" H 7650 2900 50  0000 C CNN
 F 2 "" H 7650 3050 50  0001 C CNN
@@
 	0    -1   -1   0
 $EndComp
-$Comp
-L L298 U9
-U 1 1 5A0B4B28
-P 5250 2700
-F 0 "U9" H 5250 2700 60  0000 C CNN
-F 1 "L298" H 5250 2800 60  0000 C CNN
-F 2 "L298P:SOIC127P1420X360-21N" H 5450 3300 60  0000 C CNN
-F 3 "" H 5250 2700 60  0001 C CNN
-	1    5250 2700
-	1    0    0    -1
-$EndComp
-Wire Wire Line
-	3950 2500 4400 2500
-Wire Wire Line
-	3775 2600 4400 2600
-Wire Wire Line
-	3800 2700 4400 2700
-Wire Wire Line
-	3400 2900 4400 2900
-Wire Wire Line
-	3600 2800 4400 2800
 Text Label 4150 2500 2    60   ~ 0
 OUT1
@@
 Text Label 4150 2900 2    60   ~ 0
 PWMA
-Wire Wire Line
-	3800 2700 3800 2900
-$Comp
-L GND #PWR019
-U 1 1 5A0B56EE
-P 3800 3300
-F 0 "#PWR019" H 3800 3050 50  0001 C CNN
-F 1 "GND" H 3800 3150 50  0000 C CNN
-F 2 "" H 3800 3300 50  0001 C CNN
-F 3 "" H 3800 3300 50  0001 C CNN
-	1    3800 3300
-	1    0    0    -1
-$EndComp
-Wire Wire Line
-	3800 3200 3800 3300
 $Comp
 L 74AHC1G04 U3
@@
 	1    0    0    -1
 $EndComp
-Wire Wire Line
-	4400 3000 3550 3000
-$Comp
-L GND #PWR020
+$Comp
+L GND #PWR022
 U 1 1 5A0B5AAE
 P 3050 3300
-F 0 "#PWR020" H 3050 3050 50  0001 C CNN
+F 0 "#PWR022" H 3050 3050 50  0001 C CNN
 F 1 "GND" H 3050 3150 50  0000 C CNN
 F 2 "" H 3050 3300 50  0001 C CNN
@@
 	1    0    0    -1
 $EndComp
-Wire Wire Line
-	3050 2550 3050 2800
-Wire Wire Line
-	3050 2600 2900 2600
-Connection ~ 3050 2600
 Text Label 3050 2600 0    60   ~ 0
 +5V
@@
 F 0 "C1" H 2775 2700 50  0000 L CNN
 F 1 "1uF" H 2775 2500 50  0000 L CNN
-F 2 "Capacitor_SMD:C_0805_2012Metric" H 2788 2450 50  0001 C CNN
+F 2 "Capacitors_SMD:C_0805" H 2788 2450 50  0001 C CNN
 F 3 "" H 2750 2600 50  0001 C CNN
 	1    2750 2600
@@
 $EndComp
 $Comp
-L GND #PWR021
+L GND #PWR023
 U 1 1 5A0B5C08
 P 2500 2600
-F 0 "#PWR021" H 2500 2350 50  0001 C CNN
+F 0 "#PWR023" H 2500 2350 50  0001 C CNN
 F 1 "GND" H 2500 2450 50  0000 C CNN
 F 2 "" H 2500 2600 50  0001 C CNN
@@
 	0    1    1    0
 $EndComp
-Wire Wire Line
-	2500 2600 2600 2600
-NoConn ~ 4400 2400
-NoConn ~ 6100 2400
-Wire Wire Line
-	3950 2350 3950 2500
-Wire Wire Line
-	3775 2600 3775 2350
-Wire Wire Line
-	3600 2800 3600 2350
-Wire Wire Line
-	3400 2350 3400 2900
-Wire Wire Line
-	6650 2500 6650 2350
-Wire Wire Line
-	6825 2600 6825 2350
-Wire Wire Line
-	6675 2900 6675 3000
-Wire Wire Line
-	6825 2800 6825 3000
-Wire Wire Line
-	4250 2200 4250 3300
-$Comp
-L GND #PWR022
-U 1 1 5A979197
-P 5250 3450
-F 0 "#PWR022" H 5250 3200 50  0001 C CNN
-F 1 "GND" H 5250 3300 50  0000 C CNN
-F 2 "" H 5250 3450 50  0001 C CNN
-F 3 "" H 5250 3450 50  0001 C CNN
-	1    5250 3450
-	1    0    0    -1
-$EndComp
-Wire Wire Line
-	3050 3300 3050 3200
+NoConn ~ 4450 2400
+NoConn ~ 6050 2400
 Text HLabel 3400 2350 1    60   Input ~ 0
 PWMA
@@
 DIRB
 $Comp
-L +5V #PWR023
+L +5V #PWR024
 U 1 1 5AA17AD4
 P 3050 2550
-F 0 "#PWR023" H 3050 2400 50  0001 C CNN
+F 0 "#PWR024" H 3050 2400 50  0001 C CNN
 F 1 "+5V" H 3050 2690 50  0000 C CNN
 F 2 "" H 3050 2550 50  0001 C CNN
@@
 F 0 "C7" H 3825 3150 50  0000 L CNN
 F 1 "100uF,25V" H 3825 2950 50  0000 L CNN
-F 2 "Capacitors_SMD:C_0805_HandSoldering" H 3838 2900 50  0001 C CNN
+F 2 "Capacitors_SMD:CP_Elec_6.3x5.3" H 3838 2900 50  0001 C CNN
 F 3 "" H 3800 3050 50  0001 C CNN
 	1    3800 3050
@@
 $EndComp
 $Comp
-L +5V #PWR024
+L +5V #PWR025
 U 1 1 5AA17E98
-P 6300 2050
-F 0 "#PWR024" H 6300 1900 50  0001 C CNN
-F 1 "+5V" H 6300 2190 50  0000 C CNN
-F 2 "" H 6300 2050 50  0001 C CNN
-F 3 "" H 6300 2050 50  0001 C CNN
-	1    6300 2050
-	1    0    0    -1
-$EndComp
-$Comp
-L +5V #PWR025
+P 6350 3000
+F 0 "#PWR025" H 6350 2850 50  0001 C CNN
+F 1 "+5V" H 6350 3140 50  0000 C CNN
+F 2 "" H 6350 3000 50  0001 C CNN
+F 3 "" H 6350 3000 50  0001 C CNN
+	1    6350 3000
+	-1   0    0    1
+$EndComp
+$Comp
+L +5V #PWR026
 U 1 1 5AA17EEA
 P 7150 3100
-F 0 "#PWR025" H 7150 2950 50  0001 C CNN
+F 0 "#PWR026" H 7150 2950 50  0001 C CNN
 F 1 "+5V" H 7150 3240 50  0000 C CNN
 F 2 "" H 7150 3100 50  0001 C CNN
@@
 Text HLabel 6825 2350 1    60   Input ~ 0
 OUT3
+$Comp
+L GND #PWR027
+U 1 1 5AB2A4E4
+P 5250 3600
+F 0 "#PWR027" H 5250 3350 50  0001 C CNN
+F 1 "GND" H 5250 3450 50  0000 C CNN
+F 2 "" H 5250 3600 50  0001 C CNN
+F 3 "" H 5250 3600 50  0001 C CNN
+	1    5250 3600
+	1    0    0    -1
+$EndComp
+$Comp
+L L298P IC3
+U 1 1 5AB3217D
+P 4450 2200
+F 0 "IC3" H 5900 2500 50  0000 L CNN
+F 1 "L298P" H 5900 2400 50  0000 L CNN
+F 2 "L298Poud:SOIC127P1420X360-21N" H 5900 2300 50  0001 L CNN
+F 3 "http://docs-europe.electrocomponents.com/webdocs/135f/0900766b8135fb62.pdf" H 5900 2200 50  0001 L CNN
+F 4 "L298P, Full Bridge Motor Driver, 3A Dual Full Bridge Motor Driver,, 25W 4.8  46 V, 20-Pin Power SO" H 5900 2100 50  0001 L CNN "Description"
+F 5 "3.6" H 5900 2000 50  0001 L CNN "Height"
+F 6 "STMicroelectronics" H 5900 1900 50  0001 L CNN "Manufacturer_Name"
+F 7 "L298P" H 5900 1800 50  0001 L CNN "Manufacturer_Part_Number"
+F 8 "7147715P" H 5900 1700 50  0001 L CNN "RS Part Number"
+F 9 "http://uk.rs-online.com/web/p/products/7147715P" H 5900 1600 50  0001 L CNN "RS Price/Stock"
+F 10 "70013871" H 5900 1500 50  0001 L CNN "Allied_Number"
+F 11 "http://www.alliedelec.com/stmicroelectronics-l298p/70013871/" H 5900 1400 50  0001 L CNN "Allied Price/Stock"
+	1    4450 2200
+	1    0    0    -1
+$EndComp
+Wire Wire Line
+	6050 2500 6650 2500
+Wire Wire Line
+	6050 2600 6825 2600
+Wire Wire Line
+	6050 2800 6825 2800
+Wire Wire Line
+	6050 2900 6675 2900
+Wire Wire Line
+	6050 2700 6650 2700
+Wire Wire Line
+	7150 2900 7150 3100
+Wire Wire Line
+	7150 3050 7350 3050
+Connection ~ 7150 3050
+Wire Wire Line
+	3950 2500 4450 2500
+Wire Wire Line
+	3775 2600 4450 2600
+Wire Wire Line
+	3800 2700 4450 2700
+Wire Wire Line
+	3400 2900 4450 2900
+Wire Wire Line
+	3600 2800 4450 2800
+Wire Wire Line
+	3800 2700 3800 2900
+Wire Wire Line
+	3800 3200 3800 3300
+Wire Wire Line
+	3550 3000 4450 3000
+Wire Wire Line
+	3050 2550 3050 2800
+Wire Wire Line
+	3050 2600 2900 2600
+Connection ~ 3050 2600
+Wire Wire Line
+	2500 2600 2600 2600
+Wire Wire Line
+	3950 2350 3950 2500
+Wire Wire Line
+	3775 2600 3775 2350
+Wire Wire Line
+	3600 2800 3600 2350
+Wire Wire Line
+	3400 2350 3400 2900
+Wire Wire Line
+	6650 2500 6650 2350
+Wire Wire Line
+	6825 2600 6825 2350
+Wire Wire Line
+	6675 2900 6675 3000
+Wire Wire Line
+	6825 2800 6825 3000
+Wire Wire Line
+	3050 3300 3050 3200
+Wire Wire Line
+	6050 3100 6250 3100
+Wire Wire Line
+	6250 2200 6250 3300
+Wire Wire Line
+	6050 2200 6250 2200
+Connection ~ 6250 3100
+Wire Wire Line
+	6050 2300 6250 2300
+Connection ~ 6250 2300
+Wire Wire Line
+	6050 3000 6350 3000
+Wire Wire Line
+	4250 3300 4250 2200
+Wire Wire Line
+	4250 2200 4450 2200
+Wire Wire Line
+	4450 2300 4250 2300
+Connection ~ 4250 2300
+Wire Wire Line
+	4450 3100 4250 3100
+Connection ~ 4250 3100
+Wire Wire Line
+	7150 2500 7150 2450
+$Comp
+L GND #PWR028
+U 1 1 5AB43D0E
+P 3800 3300
+F 0 "#PWR028" H 3800 3050 50  0001 C CNN
+F 1 "GND" H 3800 3150 50  0000 C CNN
+F 2 "" H 3800 3300 50  0001 C CNN
+F 3 "" H 3800 3300 50  0001 C CNN
+	1    3800 3300
+	1    0    0    -1
+$EndComp
 $EndSCHEMATC

Commit message: verbeteringen kicad
Changed lines of the file:
@@
 Comment4 ""
 $EndDescr
-$Comp
-L GND #PWR014
-U 1 1 5A0B4BA1
-P 4250 3300
-F 0 "#PWR014" H 4250 3050 50  0001 C CNN
-F 1 "GND" H 4250 3150 50  0000 C CNN
-F 2 "" H 4250 3300 50  0001 C CNN
-F 3 "" H 4250 3300 50  0001 C CNN
-	1    4250 3300
-	1    0    0    -1
-$EndComp
-$Comp
-L GND #PWR015
-U 1 1 5A0B4C37
-P 6250 3300
-F 0 "#PWR015" H 6250 3050 50  0001 C CNN
-F 1 "GND" H 6250 3150 50  0000 C CNN
-F 2 "" H 6250 3300 50  0001 C CNN
-F 3 "" H 6250 3300 50  0001 C CNN
-	1    6250 3300
-	1    0    0    -1
-$EndComp
 Text Label 6350 2500 0    60   ~ 0
 OUT4
@@
 $EndComp
 $Comp
-L GND #PWR016
-U 1 1 5A0B4D89
-P 7150 2450
-F 0 "#PWR016" H 7150 2200 50  0001 C CNN
-F 1 "GND" H 7150 2300 50  0000 C CNN
-F 2 "" H 7150 2450 50  0001 C CNN
-F 3 "" H 7150 2450 50  0001 C CNN
-	1    7150 2450
-	-1   0    0    1
-$EndComp
-$Comp
 L C C8
 U 1 1 5A0B4FB6
@@
 	0    1    1    0
 $EndComp
-$Comp
-L GND #PWR017
-U 1 1 5A0B5004
-P 7650 3050
-F 0 "#PWR017" H 7650 2800 50  0001 C CNN
-F 1 "GND" H 7650 2900 50  0000 C CNN
-F 2 "" H 7650 3050 50  0001 C CNN
-F 3 "" H 7650 3050 50  0001 C CNN
-	1    7650 3050
-	0    -1   -1   0
-$EndComp
 Text Label 4150 2500 2    60   ~ 0
 OUT1
@@
 F 3 "" H 3100 3000 50  0001 C CNN
 	1    3100 3000
-	1    0    0    -1
-$EndComp
-$Comp
-L GND #PWR018
-U 1 1 5A0B5AAE
-P 3050 3300
-F 0 "#PWR018" H 3050 3050 50  0001 C CNN
-F 1 "GND" H 3050 3150 50  0000 C CNN
-F 2 "" H 3050 3300 50  0001 C CNN
-F 3 "" H 3050 3300 50  0001 C CNN
-	1    3050 3300
 	1    0    0    -1
 $EndComp
@@
 Text HLabel 6825 2350 1    60   Input ~ 0
 OUT3
-$Comp
-L GND #PWR023
-U 1 1 5AB2A4E4
-P 5250 3600
-F 0 "#PWR023" H 5250 3350 50  0001 C CNN
-F 1 "GND" H 5250 3450 50  0000 C CNN
-F 2 "" H 5250 3600 50  0001 C CNN
-F 3 "" H 5250 3600 50  0001 C CNN
-	1    5250 3600
-	1    0    0    -1
-$EndComp
 $Comp
 L L298P IC3
@@
 Wire Wire Line
 	7150 2500 7150 2450
-$Comp
-L GND #PWR024
-U 1 1 5AB43D0E
-P 3800 3300
-F 0 "#PWR024" H 3800 3050 50  0001 C CNN
-F 1 "GND" H 3800 3150 50  0000 C CNN
-F 2 "" H 3800 3300 50  0001 C CNN
-F 3 "" H 3800 3300 50  0001 C CNN
-	1    3800 3300
-	1    0    0    -1
-$EndComp
+Text HLabel 7150 2450 0    60   Input ~ 0
+GND
+Text HLabel 7650 3050 2    60   Input ~ 0
+GND
+Text HLabel 6250 3300 2    60   Input ~ 0
+GND
+Text HLabel 5250 3600 2    60   Input ~ 0
+GND
+Text HLabel 4250 3300 2    60   Input ~ 0
+GND
+Text HLabel 3800 3300 2    60   Input ~ 0
+GND
+Text HLabel 3050 3300 2    60   Input ~ 0
+GND
 $EndSCHEMATC

Commit message: PCBtotaal
Parts:
- C1: value 1uF -> 0.11uF
Changed lines of the file:
@@
 P 2750 2600
 F 0 "C1" H 2775 2700 50  0000 L CNN
-F 1 "1uF" H 2775 2500 50  0000 L CNN
+F 1 "0.11uF" H 2775 2500 50  0000 L CNN
 F 2 "Capacitors_SMD:C_0805" H 2788 2450 50  0001 C CNN
 F 3 "" H 2750 2600 50  0001 C CNN
@@
 $EndComp
 $Comp
-L GND #PWR019
+L GND #PWR03
 U 1 1 5A0B5C08
 P 2500 2600
-F 0 "#PWR019" H 2500 2350 50  0001 C CNN
+F 0 "#PWR03" H 2500 2350 50  0001 C CNN
 F 1 "GND" H 2500 2450 50  0000 C CNN
 F 2 "" H 2500 2600 50  0001 C CNN
@@
 DIRB
 $Comp
-L +5V #PWR020
+L +5V #PWR04
 U 1 1 5AA17AD4
 P 3050 2550
-F 0 "#PWR020" H 3050 2400 50  0001 C CNN
+F 0 "#PWR04" H 3050 2400 50  0001 C CNN
 F 1 "+5V" H 3050 2690 50  0000 C CNN
 F 2 "" H 3050 2550 50  0001 C CNN
@@
 $EndComp
 $Comp
-L +5V #PWR021
+L +5V #PWR05
 U 1 1 5AA17E98
 P 6350 3000
-F 0 "#PWR021" H 6350 2850 50  0001 C CNN
+F 0 "#PWR05" H 6350 2850 50  0001 C CNN
 F 1 "+5V" H 6350 3140 50  0000 C CNN
 F 2 "" H 6350 3000 50  0001 C CNN
@@
 $EndComp
 $Comp
-L +5V #PWR022
+L +5V #PWR06
 U 1 1 5AA17EEA
 P 7150 3100
-F 0 "#PWR022" H 7150 2950 50  0001 C CNN
+F 0 "#PWR06" H 7150 2950 50  0001 C CNN
 F 1 "+5V" H 7150 3240 50  0000 C CNN
 F 2 "" H 7150 3100 50  0001 C CNN
